Commit message: THROWING

File: urdf/ur5.urdf (robot description, URDF)
Before this commit: robot sisbot, 11 links, 10 joints
Joints:
- joint left_gripper_motor: limit lower=-0.00 upper=0.04 effort=10.0 velocity=100 -> lower=-0.00 upper=0.04 effort=10.0 velocity=1000; origin xyz=-0.05 0.1 0.005 rpy=-1.57 0.0 0.0 -> xyz=-0.06 0.1 0.005 rpy=-1.57 0.0 0.0
- joint right_gripper_motor: limit lower=-0.04 upper=0.0 effort=10.0 velocity=100 -> lower=-0.04 upper=0.0 effort=10.0 velocity=1000; origin xyz=0.05 0.1 -0.005 rpy=-1.57 0.0 0.0 -> xyz=0.06 0.1 -0.005 rpy=-1.57 0.0 0.0
